Commit message: Fix robot instability and gazebo shaking

File: src/waste_sorting_description/urdf/waste_robot.urdf (robot description, URDF)
Before this commit: robot waste_robot, 5 links, 4 joints
Links:
- link base_link: geometry visual box size=0.5 0.5 0.1
Joints:
- joint elbow_joint: type revolute -> fixed
- joint fixed: origin (none) -> xyz=0 0 0 rpy=0 0 0
- joint shoulder_joint: type revolute -> fixed
